Commit message: Created a diffrential drive robot model in gazebo with its plugins for camera and lidar

File: src/robot_description/urdf/robot.urdf.xacro (robot description, xacro)
@@ -3,5 +3,5 @@
        xmlns:xacro="http://www.ros.org/wiki/xacro">
   <!-- ==================== PROPERTIES ==================== -->
-  <xacro:property name="base_length" value="0.3"/>
+  <xacro:property name="base_length" value="0.25"/>
   <xacro:property name="base_width"  value="0.2"/>
   <xacro:property name="base_height" value="0.1"/>
@@ -74,8 +74,9 @@
                               h="${wheel_width}"/>
     </link>
-    <joint name="${name}_wheel_joint" type="continuous">
+    <joint name="${name}_wheel_joint" type="revolute">
       <parent link="base_link"/>
       <child link="${name}_wheel"/>
-      <origin xyz="0 ${y_offset} 0" rpy="-1.5707 0 0"/>
+      <origin xyz="-0.05 ${y_offset} -0.05" rpy="-1.5707 0 0"/>
+      <limit lower="-1e+16" upper="1e+16" effort="10" velocity="10"/>
       <axis xyz="0 0 1"/>
     </joint>
@@ -183,3 +184,67 @@
     <origin xyz="0.15 0 0.05" rpy="0 -0.523 0"/>
   </joint>
+<gazebo>
+	<plugin filename="gz-sim-diff-drive-system" name="gz::sim::systems::DiffDrive">
+		<left_joint>left_wheel_joint</left_joint>
+		<right_joint>right_wheel_joint</right_joint>
+		<wheel_seperation>0.24</wheel_seperation>
+		<wheel_radius>0.05</wheel_radius>
+		<odom_publish_frequency>10</odom_publish_frequency>
+		<topic>/model/my_robot/cmd_vel</topic>
+		<odom_topic>model/my_robot/odom</odom_topic>
+		<frame_id>odom</frame_id>
+		<child_frame_id>base_link</child_frame_id>
+	</plugin>
+</gazebo>
+<gazebo reference="lidar_link">
+  <sensor name="lidar" type="gpu_lidar">
+    <topic>/scan</topic>
+    <update_rate>10</update_rate>
+    <lidar>
+      <scan>
+        <horizontal>
+          <samples>360</samples>
+          <resolution>1</resolution>
+          <min_angle>-3.14159</min_angle>
+          <max_angle>3.14159</max_angle>
+        </horizontal>
+      </scan>
+      <range>
+        <min>0.12</min>
+        <max>10.0</max>
+        <resolution>0.01</resolution>
+      </range>
+    </lidar>
+    <always_on>1</always_on>
+    <visualize>true</visualize>
+  </sensor>
+</gazebo>
+<gazebo reference="base_link">
+  <sensor name="imu_sensor" type="imu">
+    <always_on>1</always_on>
+    <update_rate>100</update_rate>
+    <topic>/imu</topic>
+    <visualize>true</visualize>
+  </sensor>
+</gazebo>
+<gazebo reference="camera_link">
+  <sensor name="camera" type="camera">
+    <topic>/camera/image_raw</topic>
+    <update_rate>30</update_rate>
+    <camera>
+      <horizontal_fov>1.3962634</horizontal_fov>
+      <image>
+        <width>640</width>
+        <height>480</height>
+        <format>R8G8B8</format>
+      </image>
+      <clip>
+        <near>0.02</near>
+        <far>300</far>
+      </clip>
+    </camera>
+    <always_on>1</always_on>
+    <visualize>true</visualize>
+  </sensor>
+</gazebo>
 </robot>

Commit message: Redesign: Complete redesigning of AMR robot, changed it 4 wheeled lowered the body height and added an arm mount also changed themounting position of lidar.

File: src/robot_description/urdf/robot.urdf.xacro (robot description, xacro)
@@ -3,8 +3,8 @@
        xmlns:xacro="http://www.ros.org/wiki/xacro">
   <!-- ==================== PROPERTIES ==================== -->
-  <xacro:property name="base_length" value="0.25"/>
-  <xacro:property name="base_width"  value="0.2"/>
-  <xacro:property name="base_height" value="0.1"/>
-  <xacro:property name="base_mass"   value="2.0"/>
+  <xacro:property name="base_length" value="0.35"/>
+  <xacro:property name="base_width"  value="0.25"/>
+  <xacro:property name="base_height" value="0.07"/>
+  <xacro:property name="base_mass"   value="2.5"/>
   <xacro:property name="wheel_radius" value="0.05"/>
   <xacro:property name="wheel_width"  value="0.04"/>
@@ -53,5 +53,5 @@
   </xacro:macro>
   <!-- ==================== WHEEL MACRO ==================== -->
-  <xacro:macro name="wheel" params="name y_offset">
+  <xacro:macro name="wheel" params="name x_offset y_offset">
     <link name="${name}_wheel">
       <visual>
@@ -77,5 +77,5 @@
       <parent link="base_link"/>
       <child link="${name}_wheel"/>
-      <origin xyz="-0.05 ${y_offset} -0.05" rpy="-1.5707 0 0"/>
+      <origin xyz="${x_offset} ${y_offset} -0.035" rpy="-1.5707 0 0"/>
       <limit lower="-1e+16" upper="1e+16" effort="10" velocity="10"/>
       <axis xyz="0 0 1"/>
@@ -104,32 +104,45 @@
                        z="${base_height}"/>
   </link>
+  <!-- ==================== Cover_plate ==================== -->
+  <link name="cover_plate">
+  <visual>
+    <origin xyz="0 0 0" rpy="0 0 0"/>
+    <geometry>
+      <box size="0.35 0.30 0.01"/>
+    </geometry>
+    <material name="dark_grey">
+      <color rgba="0.2 0.2 0.2 1"/>
+    </material>
+  </visual>
+  <xacro:box_inertia m="0.3" x="0.35" y="0.30" z="0.01"/>
+</link>
+<joint name="cover_plate_joint" type="fixed">
+  <parent link="base_link"/>
+  <child link="cover_plate"/>
+  <origin xyz="0 0 0.040" rpy="0 0 0"/>
+</joint>
+<!-- ==================== Arm_Mount ==================== -->
+<link name="arm_mount">
+  <visual>
+    <origin xyz="0 0 0" rpy="0 0 0"/>
+    <geometry>
+      <cylinder radius="0.04" length="0.045"/>
+    </geometry>
+    <material name="dark_grey">
+      <color rgba="0.2 0.2 0.2 1"/>
+    </material>
+  </visual>
+  <xacro:cylinder_inertia m="0.3" r="0.04" h="0.045"/>
+</link>
+<joint name="arm_mount_joint" type="fixed">
+  <parent link="base_link"/>
+  <child link="arm_mount"/>
+  <origin xyz="0.0 0 0.07" rpy="0 0 0"/>
+</joint>
   <!-- ==================== WHEELS ==================== -->
-  <xacro:wheel name="left"  y_offset="0.12"/>
-  <xacro:wheel name="right" y_offset="-0.12"/>
-  <!-- ==================== CASTER WHEEL ==================== -->
-  <link name="caster_link">
-    <visual>
-      <origin xyz="0 0 0" rpy="0 0 0"/>
-      <geometry>
-        <sphere radius="${caster_radius}"/>
-      </geometry>
-      <material name="red">
-        <color rgba="0.8 0 0 1"/>
-      </material>
-    </visual>
-    <collision>
-      <origin xyz="0 0 0" rpy="0 0 0"/>
-      <geometry>
-        <sphere radius="${caster_radius}"/>
-      </geometry>
-    </collision>
-    <xacro:sphere_inertia m="${caster_mass}" r="${caster_radius}"/>
-  </link>
-  <joint name="caster_joint" type="fixed">
-    <parent link="base_link"/>
-    <child link="caster_link"/>
-    <!-- Front of robot, below base center -->
-    <origin xyz="0.1 0 -0.05" rpy="0 0 0"/>
-  </joint>
+  <xacro:wheel name="front_left" x_offset="0.12" y_offset="0.14"/>
+  <xacro:wheel name="front_right" x_offset="0.12" y_offset="-0.14"/>
+  <xacro:wheel name="rear_left"   x_offset="-0.12" y_offset="0.14"/>
+  <xacro:wheel name="rear_right"  x_offset="-0.12" y_offset="-0.14"/>
   <!-- ==================== LIDAR ==================== -->
   <link name="lidar_link">
@@ -157,5 +170,5 @@
     <child link="lidar_link"/>
     <!-- On top of base, centered -->
-    <origin xyz="0 0 0.075" rpy="0 0 0"/>
+    <origin xyz="-0.12 0 0.075" rpy="0 0 0"/>
   </joint>
   <!-- ==================== CAMERA ==================== -->
@@ -182,11 +195,11 @@
     <child link="camera_link"/>
     <!-- Front of robot, tilted down 30 degrees -->
-    <origin xyz="0.15 0 0.05" rpy="0 -0.523 0"/>
+    <origin xyz="0.175 0 0.04" rpy="0 -0.523 0"/>
   </joint>
 <gazebo>
 	<plugin filename="gz-sim-diff-drive-system" name="gz::sim::systems::DiffDrive">
-		<left_joint>left_wheel_joint</left_joint>
-		<right_joint>right_wheel_joint</right_joint>
-		<wheel_separation>0.24</wheel_separation>
+		<left_joint>front_left_wheel_joint</left_joint>
+		<right_joint>front_right_wheel_joint</right_joint>
+		<wheel_separation>0.28</wheel_separation>
 		<wheel_radius>0.05</wheel_radius>
 		<odom_publish_frequency>10</odom_publish_frequency>
