Commit message: Added a new waypoint navigation node

File: src/robot_description/urdf/robot.urdf.xacro (robot description, xacro)
@@ -122,22 +122,4 @@
   <origin xyz="0 0 0.040" rpy="0 0 0"/>
 </joint>
-<!-- ==================== Arm_Mount ==================== -->
-<link name="arm_mount">
-  <visual>
-    <origin xyz="0 0 0" rpy="0 0 0"/>
-    <geometry>
-      <cylinder radius="0.04" length="0.045"/>
-    </geometry>
-    <material name="dark_grey">
-      <color rgba="0.2 0.2 0.2 1"/>
-    </material>
-  </visual>
-  <xacro:cylinder_inertia m="0.3" r="0.04" h="0.045"/>
-</link>
-<joint name="arm_mount_joint" type="fixed">
-  <parent link="base_link"/>
-  <child link="arm_mount"/>
-  <origin xyz="0.0 0 0.07" rpy="0 0 0"/>
-</joint>
   <!-- ==================== WHEELS ==================== -->
   <xacro:wheel name="front_left" x_offset="0.12" y_offset="0.14"/>
@@ -170,5 +152,5 @@
     <child link="lidar_link"/>
     <!-- On top of base, centered -->
-    <origin xyz="-0.12 0 0.075" rpy="0 0 0"/>
+    <origin xyz="0.0 0 0.07" rpy="0 0 0"/>
   </joint>
   <!-- ==================== CAMERA ==================== -->
@@ -211,5 +193,5 @@
 </gazebo>
 <gazebo reference="lidar_link">
-  <sensor name="lidar" type="gpu_lidar">
+  <sensor name="lidar" type="lidar">
     <topic>/scan</topic>
     <update_rate>10</update_rate>
@@ -261,4 +243,4 @@
   </sensor>
 </gazebo>
-<xacro:include filename="$(find arm_description)/urdf/arm.urdf.xacro"/>
+<!-- <xacro:include filename="$(find arm_description)/urdf/arm.urdf.xacro"/> -->
 </robot>

Commit message: Added a multiroom pick and place enviroment for the version 2.0

File: src/robot_description/urdf/robot.urdf.xacro (robot description, xacro)
@@ -74,12 +74,24 @@
                               h="${wheel_width}"/>
     </link>
-    <joint name="${name}_wheel_joint" type="revolute">
+    <joint name="${name}_wheel_joint" type="continuous">
       <parent link="base_link"/>
       <child link="${name}_wheel"/>
       <origin xyz="${x_offset} ${y_offset} -0.035" rpy="-1.5707 0 0"/>
-      <limit lower="-1e+16" upper="1e+16" effort="10" velocity="10"/>
       <axis xyz="0 0 1"/>
     </joint>
-  </xacro:macro>
+    <gazebo reference="${name}_wheel">
+      <mu1>1.0</mu1>
+      <mu2>1.0</mu2>
+      <kp>1000000.0</kp>
+      <kd>1.0</kd>
+    </gazebo>
+  </xacro:macro>
+  <!-- ==================== BASE FOOTPRINT ==================== -->
+  <link name="base_footprint"/>
+  <joint name="base_footprint_joint" type="fixed">
+    <parent link="base_footprint"/>
+    <child link="base_link"/>
+    <origin xyz="0 0 0.085" rpy="0 0 0"/>
+  </joint>
   <!-- ==================== BASE LINK ==================== -->
   <link name="base_link">
@@ -180,20 +192,33 @@
   </joint>
 <gazebo>
-	<plugin filename="gz-sim-diff-drive-system" name="gz::sim::systems::DiffDrive">
-		<left_joint>front_left_wheel_joint</left_joint>
-		<right_joint>front_right_wheel_joint</right_joint>
-		<wheel_separation>0.28</wheel_separation>
-		<wheel_radius>0.05</wheel_radius>
-		<odom_publish_frequency>10</odom_publish_frequency>
-		<topic>/model/my_robot/cmd_vel</topic>
-		<odom_topic>/model/my_robot/odometry</odom_topic>
-		<frame_id>odom</frame_id>
-		<child_frame_id>base_link</child_frame_id>
-	</plugin>
+  <plugin filename="gz-sim-diff-drive-system" name="gz::sim::systems::DiffDrive">
+    <left_joint>front_left_wheel_joint</left_joint>
+    <left_joint>rear_left_wheel_joint</left_joint>
+    <right_joint>front_right_wheel_joint</right_joint>
+    <right_joint>rear_right_wheel_joint</right_joint>
+    <wheel_separation>0.28</wheel_separation>
+    <wheel_radius>0.05</wheel_radius>
+    <odom_publish_frequency>20</odom_publish_frequency>
+    <topic>/model/my_robot/cmd_vel</topic>
+    <odom_topic>/model/my_robot/odometry</odom_topic>
+    <frame_id>odom</frame_id>
+    <child_frame_id>base_footprint</child_frame_id>
+  </plugin>
+  <plugin filename="gz-sim-joint-state-publisher-system" name="gz::sim::systems::JointStatePublisher">
+    <update_rate>20</update_rate>
+    <topic>/joint_states</topic>
+    <joint_name>front_left_wheel_joint</joint_name>
+    <joint_name>front_right_wheel_joint</joint_name>
+    <joint_name>rear_left_wheel_joint</joint_name>
+    <joint_name>rear_right_wheel_joint</joint_name>
+  </plugin>
 </gazebo>
 <gazebo reference="lidar_link">
-  <sensor name="lidar" type="lidar">
+  <sensor name="lidar" type="gpu_lidar">
     <topic>/scan</topic>
     <update_rate>10</update_rate>
+    <gz_frame_id>lidar_link</gz_frame_id>
+    <frame_id>lidar_link</frame_id>
+    <ignition_frame_id>lidar_link</ignition_frame_id>
     <lidar>
       <scan>
@@ -220,4 +245,7 @@
     <update_rate>100</update_rate>
     <topic>/imu</topic>
+    <gz_frame_id>base_link</gz_frame_id>
+    <frame_id>base_link</frame_id>
+    <ignition_frame_id>base_link</ignition_frame_id>
     <visualize>true</visualize>
   </sensor>
@@ -226,4 +254,7 @@
   <sensor name="camera" type="camera">
     <topic>/camera/image_raw</topic>
+    <gz_frame_id>camera_link</gz_frame_id>
+    <frame_id>camera_link</frame_id>
+    <ignition_frame_id>camera_link</ignition_frame_id>
     <update_rate>30</update_rate>
     <camera>
@@ -243,4 +274,3 @@
   </sensor>
 </gazebo>
-<!-- <xacro:include filename="$(find arm_description)/urdf/arm.urdf.xacro"/> -->
 </robot>

Commit message: Added aruco_markers and aruco_marker_detection node for arm detection.

File: src/robot_description/urdf/robot.urdf.xacro (robot description, xacro)
@@ -283,6 +283,9 @@
     <origin xyz="0.0 0 0.030" rpy="0 0 0"/>
   </joint>
-  <!-- ==================== CAMERA ==================== -->
-  <link name="camera_link">
+  <!-- ==================== CAMERA FRONT ====================
+       Faces forward (+X), tilted down 30° to see floor/markers on approach.
+       Topic: /camera/front/image_raw
+  -->
+  <link name="camera_link_1">
     <visual>
       <origin xyz="0 0 0" rpy="0 0 0"/>
@@ -302,9 +305,39 @@
     <xacro:box_inertia m="0.1" x="0.05" y="0.05" z="0.03"/>
   </link>
-  <joint name="camera_joint" type="fixed">
+  <joint name="camera_joint_1" type="fixed">
     <parent link="base_link"/>
-    <child link="camera_link"/>
-    <!-- Front of robot, tilted down 30 degrees -->
+    <child link="camera_link_1"/>
+    <!-- Front face of robot (base_length/2=0.175), same height as cover_plate top -->
     <origin xyz="0.175 0 0.04" rpy="0 -0.523 0"/>
+  </joint>
+  <!-- ==================== CAMERA REAR ====================
+       Faces backward (-X), tilted down ~20° to see shelf-face ArUco markers
+       during reverse docking. Yaw=π flips the camera 180°; pitch=+0.349
+       produces a downward look in world frame (tilt direction inverts with yaw).
+       Topic: /camera/rear/image_raw
+  -->
+  <link name="camera_link_2">
+    <visual>
+      <origin xyz="0 0 0" rpy="0 0 0"/>
+      <geometry>
+        <box size="0.05 0.05 0.03"/>
+      </geometry>
+      <material name="orange">
+        <color rgba="1.0 0.5 0.0 1"/>
+      </material>
+    </visual>
+    <collision>
+      <origin xyz="0 0 0" rpy="0 0 0"/>
+      <geometry>
+        <box size="0.05 0.05 0.03"/>
+      </geometry>
+    </collision>
+    <xacro:box_inertia m="0.1" x="0.05" y="0.05" z="0.03"/>
+  </link>
+  <joint name="camera_joint_2" type="fixed">
+    <parent link="base_link"/>
+    <child link="camera_link_2"/>
+    <!-- Rear face of robot (x=-0.175), yaw=π faces backward, pitch=+0.349 tilts down ~20° -->
+    <origin xyz="-0.175 0 0.04" rpy="0 0.349 3.14159"/>
   </joint>
 <gazebo>
@@ -368,10 +401,33 @@
   </sensor>
 </gazebo>
-<gazebo reference="camera_link">
-  <sensor name="camera" type="camera">
-    <topic>/camera/image_raw</topic>
-    <gz_frame_id>camera_link</gz_frame_id>
-    <frame_id>camera_link</frame_id>
-    <ignition_frame_id>camera_link</ignition_frame_id>
+<gazebo reference="camera_link_1">
+  <sensor name="camera_front" type="camera">
+    <topic>/camera/front/image_raw</topic>
+    <gz_frame_id>camera_link_1</gz_frame_id>
+    <frame_id>camera_link_1</frame_id>
+    <ignition_frame_id>camera_link_1</ignition_frame_id>
+    <update_rate>30</update_rate>
+    <camera>
+      <horizontal_fov>1.3962634</horizontal_fov>
+      <image>
+        <width>640</width>
+        <height>480</height>
+        <format>R8G8B8</format>
+      </image>
+      <clip>
+        <near>0.02</near>
+        <far>300</far>
+      </clip>
+    </camera>
+    <always_on>1</always_on>
+    <visualize>true</visualize>
+  </sensor>
+</gazebo>
+<gazebo reference="camera_link_2">
+  <sensor name="camera_rear" type="camera">
+    <topic>/camera/rear/image_raw</topic>
+    <gz_frame_id>camera_link_2</gz_frame_id>
+    <frame_id>camera_link_2</frame_id>
+    <ignition_frame_id>camera_link_2</ignition_frame_id>
     <update_rate>30</update_rate>
     <camera>

Commit message: Major revamp: Added SLAM and NAV2 based path planning and moveit pick_and_place of box on the bot. Added and updated readmes for workspace and all folders.

File: src/robot_description/urdf/robot.urdf.xacro (robot description, xacro)
@@ -107,13 +107,10 @@
       <origin xyz="${x_offset} ${y_offset} -0.035" rpy="-1.5707 0 0"/>
       <axis xyz="0 0 1"/>
-      <dynamics damping="0.05" friction="0.1"/>
+      <dynamics damping="0.001" friction="0.0"/>
     </joint>
     <gazebo reference="${name}_wheel">
-      <!-- mu1/mu2 tuning for 4-fixed-wheel skid-steer:
-           mu2 too high -> bot cannot pivot (wheels scrub, chassis stalls);
-           mu2 too low  -> bot SLIDES sideways during turns (odometry lies).
-           0.3 = compromise: pivots with moderate scrub. Verified live. -->
       <mu1>1.1</mu1>
-      <mu2>0.3</mu2>
+      <mu2>0.05</mu2>
+      <fdir1>1 0 0</fdir1>
       <kp>100000.0</kp>
       <kd>10.0</kd>
@@ -435,9 +432,15 @@
     <wheel_separation>0.28</wheel_separation>
     <wheel_radius>0.05</wheel_radius>
+    <topic>/model/my_robot/cmd_vel</topic>
+    <odom_publish_frequency>0</odom_publish_frequency>
+    <odom_topic>/model/my_robot/diff_drive_unused_odom</odom_topic>
+    <tf_topic>/model/my_robot/diff_drive_unused_tf</tf_topic>
+  </plugin>
+  <plugin filename="gz-sim-odometry-publisher-system" name="gz::sim::systems::OdometryPublisher">
+    <odom_frame>odom</odom_frame>
+    <robot_base_frame>base_footprint</robot_base_frame>
+    <odom_topic>/model/my_robot/odometry</odom_topic>
     <odom_publish_frequency>20</odom_publish_frequency>
-    <topic>/model/my_robot/cmd_vel</topic>
-    <odom_topic>/model/my_robot/odometry</odom_topic>
-    <frame_id>odom</frame_id>
-    <child_frame_id>base_footprint</child_frame_id>
+    <dimensions>2</dimensions>
   </plugin>
   <plugin filename="gz-sim-joint-state-publisher-system" name="gz::sim::systems::JointStatePublisher">
@@ -467,5 +470,5 @@
       </scan>
       <range>
-        <min>0.12</min>
+        <min>0.25</min>
         <max>10.0</max>
         <resolution>0.01</resolution>

File: src/robotic_4dof_arm/urdf/arm.urdf.xacro (robot description, xacro)
@@ -81,20 +81,20 @@
   </joint>
   <link name="arm_base_link">
-    <visual>
-      <origin xyz="0 0 0" rpy="0 0 0"/>
-      <geometry>
-        <cylinder radius="${arm_base_link_radius}" length="${arm_base_link_height}"/>
-      </geometry>
-      <material name="black">
-        <color rgba="0.1 0.1 0.1 1"/>
-      </material>
-    </visual>
-    <collision>
-      <origin xyz="0 0 0" rpy="0 0 0"/>
-      <geometry>
-        <cylinder radius="0.05" length="0.02"/>
-      </geometry>
-    </collision>
-    <xacro:cylinder_inertia m="${arm_base_link_weight}" r="${arm_base_link_radius}" h="${arm_base_link_height}"/>
+  <visual>
+    <origin xyz="0 0 0" rpy="0 0 0"/>
+    <geometry>
+      <cylinder radius="${arm_base_link_radius}" length="${arm_base_link_height}"/>
+    </geometry>
+    <material name="black">
+      <color rgba="0.1 0.1 0.1 1"/>
+    </material>
+  </visual>
+  <collision>
+    <origin xyz="0 0 0" rpy="0 0 0"/>
+    <geometry>
+      <cylinder radius="0.05" length="0.02"/>
+    </geometry>
+  </collision>
+  <xacro:cylinder_inertia m="${arm_base_link_weight}" r="${arm_base_link_radius}" h="${arm_base_link_height}"/>
   </link>
   <!-- Joint 1: shoulder pan  — mounted to pedestal top -->
@@ -102,5 +102,5 @@
     <parent link="pedestal"/>
     <child link="arm_base_link"/>
-    <origin xyz="0.0 0 0.025" rpy="0 0 0"/> <!-- 0.015 (half pedestal) + 0.01 = 0.025 -->
+    <origin xyz="0.0 0 0.025" rpy="0 0 0"/>
     <limit lower="-3.14" upper="3.14" effort="150" velocity="3.14"/>
     <axis xyz="0 0 1"/>
@@ -386,61 +386,61 @@
   <!-- =================================================== -->
   <!-- ros2_control hardware interface -->
-  <ros2_control name="arm_system" type="system">
-    <hardware>
-      <plugin>gz_ros2_control/GazeboSimSystem</plugin>
-    </hardware>
-    <joint name="arm_base_joint">
-      <command_interface name="position"/>
-      <state_interface name="position">
-        <param name="initial_value">0.0</param>
-      </state_interface>
-      <state_interface name="velocity"/>
-    </joint>
-    <joint name="upper_arm_joint">
-      <command_interface name="position"/>
-      <state_interface name="position">
-        <param name="initial_value">0.0</param>
-      </state_interface>
-      <state_interface name="velocity"/>
-    </joint>
-    <joint name="forearm_joint">
-      <command_interface name="position"/>
-      <state_interface name="position">
-        <param name="initial_value">0.0</param>
-      </state_interface>
-      <state_interface name="velocity"/>
-    </joint>
-    <joint name="wrist_joint">
-      <command_interface name="position"/>
-      <state_interface name="position">
-        <param name="initial_value">0.0</param>
-      </state_interface>
-      <state_interface name="velocity"/>
-    </joint>
-    <joint name="gripper_baseTOwrist_joint">
-      <command_interface name="position"/>
-      <state_interface name="position">
-        <param name="initial_value">0.0</param>
-      </state_interface>
-      <state_interface name="velocity"/>
-    </joint>
-    <joint name="gripper_base_joint">
-      <command_interface name="position"/>
-      <state_interface name="position">
-        <param name="initial_value">0.0</param>
-      </state_interface>
-      <state_interface name="velocity"/>
-    </joint>
-    <joint name="right_prong_joint">
-      <command_interface name="position"/>
-      <state_interface name="position"/>
-      <state_interface name="velocity"/>
-    </joint>
-    <joint name="left_prong_joint">
-      <command_interface name="position"/>
-      <state_interface name="position"/>
-      <state_interface name="velocity"/>
-    </joint>
-  </ros2_control>
+<ros2_control name="arm_system" type="system">
+  <hardware>
+    <plugin>gz_ros2_control/GazeboSimSystem</plugin>
+  </hardware>
+  <joint name="arm_base_joint">
+    <command_interface name="position"/>
+    <state_interface name="position">
+      <param name="initial_value">0.0</param>
+    </state_interface>
+    <state_interface name="velocity"/>
+  </joint>
+  <joint name="upper_arm_joint">
+    <command_interface name="position"/>
+    <state_interface name="position">
+      <param name="initial_value">0.0</param>
+    </state_interface>
+    <state_interface name="velocity"/>
+  </joint>
+  <joint name="forearm_joint">
+    <command_interface name="position"/>
+    <state_interface name="position">
+      <param name="initial_value">0.0</param>
+    </state_interface>
+    <state_interface name="velocity"/>
+  </joint>
+  <joint name="wrist_joint">
+    <command_interface name="position"/>
+    <state_interface name="position">
+      <param name="initial_value">0.0</param>
+    </state_interface>
+    <state_interface name="velocity"/>
+  </joint>
+  <joint name="gripper_baseTOwrist_joint">
+    <command_interface name="position"/>
+    <state_interface name="position">
+      <param name="initial_value">0.0</param>
+    </state_interface>
+    <state_interface name="velocity"/>
+  </joint>
+  <joint name="gripper_base_joint">
+    <command_interface name="position"/>
+    <state_interface name="position">
+      <param name="initial_value">0.0</param>
+    </state_interface>
+    <state_interface name="velocity"/>
+  </joint>
+  <joint name="right_prong_joint">
+    <command_interface name="position"/>
+    <state_interface name="position"/>
+    <state_interface name="velocity"/>
+  </joint>
+  <joint name="left_prong_joint">
+    <command_interface name="position"/>
+    <state_interface name="position"/>
+    <state_interface name="velocity"/>
+  </joint>
+</ros2_control>
   <!-- ==================== GAZEBO FRICTION & CONTACT PROPERTIES ==================== -->
   <gazebo reference="right_prong_link">
@@ -460,26 +460,10 @@
     <maxVel>0.1</maxVel>
   </gazebo>
-  <!-- Path to arm_controllers.yaml — set by launch file via xacro:arg -->
-  <xacro:arg name="controllers_file" default=""/>
-  <!-- Namespace for this arm instance (arm1 or arm2) -->
-  <xacro:arg name="arm_namespace" default="arm1"/>
-  <xacro:property name="c_file" value="$(arg controllers_file)"/>
-  <!-- gz_ros2_control plugin — each instance gets its own namespace so
-       two arms can coexist with separate controller_managers -->
-  <xacro:if value="${c_file != ''}">
-    <gazebo>
-      <plugin filename="gz_ros2_control-system"
-              name="gz_ros2_control::GazeboSimROS2ControlPlugin">
-        <parameters>$(arg controllers_file)</parameters>
-        <robot_param>robot_description</robot_param>
-        <robot_param_node>arm_state_publisher</robot_param_node>
-        <ros>
-          <namespace>/$(arg arm_namespace)</namespace>
-        </ros>
-      </plugin>
-    </gazebo>
-  </xacro:if>
-  <xacro:unless value="${c_file != ''}">
-    <gazebo><static>true</static></gazebo>
-  </xacro:unless>
+<!-- gz_ros2_control plugin -->
+<gazebo>
+  <plugin filename="gz_ros2_control-system"
+          name="gz_ros2_control::GazeboSimROS2ControlPlugin">
+    <parameters>$(find robotic_4dof_arm)/config/controllers.yaml</parameters>
+  </plugin>
+</gazebo>
 </robot>
