Commit message: Updated the xacro

File: src/robot_description/urdf/robot.urdf.xacro (robot description, xacro)
@@ -15,4 +15,21 @@
   <xacro:property name="lidar_height" value="0.05"/>
   <xacro:property name="lidar_mass"   value="0.2"/>
+  <!-- Standoffs: 4 cylinders at cover_plate corners holding up standoff_floor -->
+  <xacro:property name="standoff_height" value="0.052"/>
+  <xacro:property name="standoff_radius" value="0.01"/>
+  <xacro:property name="standoff_mass"   value="0.075"/>
+  <!-- Standoff floor: same footprint as base, thin plate above standoffs -->
+  <xacro:property name="standoff_floor_length" value="0.35"/>
+  <xacro:property name="standoff_floor_width"  value="0.25"/>
+  <xacro:property name="standoff_floor_height" value="0.01"/>
+  <xacro:property name="standoff_floor_mass"   value="0.3"/>
+  <!-- Cover plate sits on top of base_link.
+       cover_plate top surface  = base_height/2 + cover_plate_joint_z + plate_half_h
+                                = 0.035 + 0.040 + 0.005 = 0.080 above base center
+       Shortcuts for pose calculations (all relative to base_link centre):
+         cover_top_z  = 0.040 + 0.005            = 0.045
+         standoff_ctr = cover_top_z + stdh/2      = 0.045 + 0.026 = 0.071
+         sfp_ctr      = cover_top_z + stdh + sfh/2= 0.045+0.052+0.005 = 0.102
+  -->
   <!-- ==================== INERTIA MACROS ==================== -->
   <xacro:macro name="box_inertia" params="m x y z">
@@ -79,11 +96,48 @@
       <origin xyz="${x_offset} ${y_offset} -0.035" rpy="-1.5707 0 0"/>
       <axis xyz="0 0 1"/>
+      <dynamics damping="0.05" friction="0.1"/>
     </joint>
     <gazebo reference="${name}_wheel">
-      <mu1>1.0</mu1>
-      <mu2>1.0</mu2>
-      <kp>1000000.0</kp>
-      <kd>1.0</kd>
+      <mu1>0.8</mu1>
+      <mu2>0.05</mu2>
+      <kp>100000.0</kp>
+      <kd>10.0</kd>
     </gazebo>
+  </xacro:macro>
+  <!-- ==================== STANDOFF MACRO ====================
+       Each standoff is a fixed cylinder connecting cover_plate to standoff_floor.
+       x_offset / y_offset place it at a corner of the plate.
+       Joint origin z = cover_plate_half_h + standoff_half_h
+                      = 0.005 + 0.026 = 0.031
+       (measured from cover_plate centre, so the bottom of the standoff
+        sits flush on the cover_plate top surface)
+  -->
+  <xacro:macro name="standoff" params="name x_offset y_offset">
+    <link name="${name}_standoff">
+      <visual>
+        <origin xyz="0 0 0" rpy="0 0 0"/>
+        <geometry>
+          <cylinder radius="${standoff_radius}" length="${standoff_height}"/>
+        </geometry>
+        <material name="silver">
+          <color rgba="0.7 0.7 0.7 1"/>
+        </material>
+      </visual>
+      <collision>
+        <origin xyz="0 0 0" rpy="0 0 0"/>
+        <geometry>
+          <cylinder radius="${standoff_radius}" length="${standoff_height}"/>
+        </geometry>
+      </collision>
+      <xacro:cylinder_inertia m="${standoff_mass}"
+                              r="${standoff_radius}"
+                              h="${standoff_height}"/>
+    </link>
+    <!-- Parent: cover_plate. z offset = plate_half_h + standoff_half_h -->
+    <joint name="${name}_standoff_joint" type="fixed">
+      <parent link="cover_plate"/>
+      <child link="${name}_standoff"/>
+      <origin xyz="${x_offset} ${y_offset} ${0.005 + standoff_height/2}" rpy="0 0 0"/>
+    </joint>
   </xacro:macro>
   <!-- ==================== BASE FOOTPRINT ==================== -->
@@ -116,28 +170,91 @@
                        z="${base_height}"/>
   </link>
-  <!-- ==================== Cover_plate ==================== -->
-  <link name="cover_plate">
-  <visual>
-    <origin xyz="0 0 0" rpy="0 0 0"/>
-    <geometry>
-      <box size="0.35 0.30 0.01"/>
-    </geometry>
-    <material name="dark_grey">
-      <color rgba="0.2 0.2 0.2 1"/>
-    </material>
-  </visual>
-  <xacro:box_inertia m="0.3" x="0.35" y="0.30" z="0.01"/>
-</link>
-<joint name="cover_plate_joint" type="fixed">
-  <parent link="base_link"/>
-  <child link="cover_plate"/>
-  <origin xyz="0 0 0.040" rpy="0 0 0"/>
-</joint>
   <!-- ==================== WHEELS ==================== -->
-  <xacro:wheel name="front_left" x_offset="0.12" y_offset="0.14"/>
-  <xacro:wheel name="front_right" x_offset="0.12" y_offset="-0.14"/>
+  <xacro:wheel name="front_left"  x_offset="0.12"  y_offset="0.14"/>
+  <xacro:wheel name="front_right" x_offset="0.12"  y_offset="-0.14"/>
   <xacro:wheel name="rear_left"   x_offset="-0.12" y_offset="0.14"/>
   <xacro:wheel name="rear_right"  x_offset="-0.12" y_offset="-0.14"/>
-  <!-- ==================== LIDAR ==================== -->
+  <!-- ==================== COVER PLATE ====================
+       Sits directly on top of base_link.
+       Joint z = base_height/2 + plate_height/2 = 0.035 + 0.005 = 0.040
+       cover_plate centre is at z=0.040 relative to base_link centre.
+       cover_plate top surface  = 0.040 + 0.005 = 0.045 above base_link centre.
+       The LiDAR mounts here.
+  -->
+  <link name="cover_plate">
+    <visual>
+      <origin xyz="0 0 0" rpy="0 0 0"/>
+      <geometry>
+        <box size="0.35 0.30 0.01"/>
+      </geometry>
+      <material name="dark_grey">
+        <color rgba="0.2 0.2 0.2 1"/>
+      </material>
+    </visual>
+    <collision>
+      <origin xyz="0 0 0" rpy="0 0 0"/>
+      <geometry>
+        <box size="0.35 0.30 0.01"/>
+      </geometry>
+    </collision>
+    <xacro:box_inertia m="0.3" x="0.35" y="0.30" z="0.01"/>
+  </link>
+  <joint name="cover_plate_joint" type="fixed">
+    <parent link="base_link"/>
+    <child link="cover_plate"/>
+    <!-- base_height/2 + cover_plate_height/2 = 0.035 + 0.005 = 0.040 -->
+    <origin xyz="0 0 0.040" rpy="0 0 0"/>
+  </joint>
+  <!-- ==================== STANDOFFS (4 corners of cover_plate) ====================
+       Corner positions: ±(base_length/2 - margin) × ±(base_width/2 - margin)
+       margin = 0.025 m keeps standoffs inside the plate footprint.
+       x: ±(0.35/2 - 0.025) = ±0.150
+       y: ±(0.25/2 - 0.025) = ±0.100
+  -->
+  <xacro:standoff name="front_left"  x_offset=" 0.150" y_offset=" 0.100"/>
+  <xacro:standoff name="front_right" x_offset=" 0.150" y_offset="-0.100"/>
+  <xacro:standoff name="rear_left"   x_offset="-0.150" y_offset=" 0.100"/>
+  <xacro:standoff name="rear_right"  x_offset="-0.150" y_offset="-0.100"/>
+  <!-- ==================== STANDOFF FLOOR ====================
+       Rests on top of all 4 standoffs.
+       Parent: cover_plate.
+       z = cover_plate_half_h + standoff_height + floor_half_h
+         = 0.005 + 0.052 + 0.005 = 0.062  (from cover_plate centre)
+       Which is 0.040 + 0.062 = 0.102 above base_link centre.
+       The delivery_box will sit on top of this floor.
+  -->
+  <link name="standoff_floor">
+    <visual>
+      <origin xyz="0 0 0" rpy="0 0 0"/>
+      <geometry>
+        <box size="${standoff_floor_length} ${standoff_floor_width} ${standoff_floor_height}"/>
+      </geometry>
+      <material name="dark_grey">
+        <color rgba="0.2 0.2 0.2 1"/>
+      </material>
+    </visual>
+    <collision>
+      <origin xyz="0 0 0" rpy="0 0 0"/>
+      <geometry>
+        <box size="${standoff_floor_length} ${standoff_floor_width} ${standoff_floor_height}"/>
+      </geometry>
+    </collision>
+    <xacro:box_inertia m="${standoff_floor_mass}"
+                       x="${standoff_floor_length}"
+                       y="${standoff_floor_width}"
+                       z="${standoff_floor_height}"/>
+  </link>
+  <joint name="standoff_floor_joint" type="fixed">
+    <parent link="cover_plate"/>
+    <child link="standoff_floor"/>
+    <!-- cover_plate_half_h + standoff_height + floor_half_h
+         = 0.005 + 0.052 + 0.005 = 0.062 -->
+    <origin xyz="0 0 0.062" rpy="0 0 0"/>
+  </joint>
+  <!-- ==================== LIDAR ====================
+       Mounts on top of cover_plate (centre of the plate).
+       Parent: cover_plate.
+       z = cover_plate_half_h + lidar_height/2 = 0.005 + 0.025 = 0.030
+  -->
   <link name="lidar_link">
     <visual>
@@ -161,8 +278,8 @@
   </link>
   <joint name="lidar_joint" type="fixed">
-    <parent link="base_link"/>
+    <parent link="cover_plate"/>
     <child link="lidar_link"/>
-    <!-- On top of base, centered -->
-    <origin xyz="0.0 0 0.07" rpy="0 0 0"/>
+    <!-- cover_plate_half_h + lidar_half_h = 0.005 + 0.025 = 0.030 -->
+    <origin xyz="0.0 0 0.030" rpy="0 0 0"/>
   </joint>
   <!-- ==================== CAMERA ==================== -->

Commit message: Added a new warehouse environment and a launch file

File: src/robot_description/urdf/arm.urdf.xacro (robot description, xacro)
@@ -61,29 +61,46 @@
     </inertial>
   </xacro:macro>
-  <!-- ==================== ARM BASE LINK ==================== -->
+  <!-- ==================== PEDESTAL & ARM BASE ==================== -->
   <link name="world"/>
+  <link name="pedestal">
+    <visual>
+      <origin xyz="0 0 0" rpy="0 0 0"/>
+      <geometry><box size="0.3 0.3 0.03"/></geometry>
+      <material name="dark_grey"><color rgba="0.2 0.2 0.2 1"/></material>
+    </visual>
+    <collision>
+      <origin xyz="0 0 0" rpy="0 0 0"/>
+      <geometry><box size="0.3 0.3 0.03"/></geometry>
+    </collision>
+    <xacro:box_inertia m="10.0" x="0.3" y="0.3" z="0.03"/>
+  </link>
+  <joint name="pedestal_joint" type="fixed">
+    <parent link="world"/>
+    <child link="pedestal"/>
+    <origin xyz="0 0 0.015" rpy="0 0 0"/>
+  </joint>
   <link name="arm_base_link">
-  <visual>
-    <origin xyz="0 0 0" rpy="0 0 0"/>
-    <geometry>
-      <cylinder radius="${arm_base_link_radius}" length="${arm_base_link_height}"/>
-    </geometry>
-    <material name="black">
-      <color rgba="0.1 0.1 0.1 1"/>
-    </material>
-  </visual>
-  <collision>
-    <origin xyz="0 0 0" rpy="0 0 0"/>
-    <geometry>
-      <cylinder radius="0.05" length="0.02"/>
-    </geometry>
-  </collision>
-  <xacro:cylinder_inertia m="${arm_base_link_weight}" r="${arm_base_link_radius}" h="${arm_base_link_height}"/>
-  </link>
-  <!-- Joint 1: shoulder pan  — d1=0.089 m up, alpha=+90 deg -->
+    <visual>
+      <origin xyz="0 0 0" rpy="0 0 0"/>
+      <geometry>
+        <cylinder radius="${arm_base_link_radius}" length="${arm_base_link_height}"/>
+      </geometry>
+      <material name="black">
+        <color rgba="0.1 0.1 0.1 1"/>
+      </material>
+    </visual>
+    <collision>
+      <origin xyz="0 0 0" rpy="0 0 0"/>
+      <geometry>
+        <cylinder radius="0.05" length="0.02"/>
+      </geometry>
+    </collision>
+    <xacro:cylinder_inertia m="${arm_base_link_weight}" r="${arm_base_link_radius}" h="${arm_base_link_height}"/>
+  </link>
+  <!-- Joint 1: shoulder pan  — mounted to pedestal top -->
   <joint name="arm_base_joint" type="revolute">
-    <parent link="world"/>
+    <parent link="pedestal"/>
     <child link="arm_base_link"/>
-    <origin xyz="0.0 0 0.01" rpy="0 0 0"/>
+    <origin xyz="0.0 0 0.025" rpy="0 0 0"/> <!-- 0.015 (half pedestal) + 0.01 = 0.025 -->
     <limit lower="-3.14" upper="3.14" effort="150" velocity="3.14"/>
     <axis xyz="0 0 1"/>
@@ -114,5 +131,5 @@
     <parent link="arm_base_link"/>
     <child link="upper_arm_link"/>
-    <origin xyz="0 0 0.01" rpy="0 -1.5707 0"/>
+    <origin xyz="0 0 0.01" rpy="0 0 0"/>
     <limit lower="-3.14" upper="3.14" effort="150" velocity="3.14"/>
     <axis xyz="0 1 0"/>
@@ -179,5 +196,5 @@
     <parent link="upper_arm_link"/>
     <child link="forearm_link"/>
-    <origin xyz="0 0 ${a2}" rpy="0 0 0"/>
+    <origin xyz="0 0 ${a2}" rpy="0 -1.5707 0"/>
     <limit lower="-3.14" upper="3.14" effort="150" velocity="3.14"/>
     <axis xyz="0 1 0"/>
@@ -226,5 +243,5 @@
     <parent link="forearm_link"/>
     <child link="wrist_link"/>
-    <origin xyz="0 0 ${a3}" rpy="1.5707 0 0"/>
+    <origin xyz="0 0 ${a3}" rpy="1.5707 -0.7854 0"/>
     <limit lower="-3.14" upper="3.14" effort="28" velocity="3.14"/>
     <axis xyz="0 0 1"/>
@@ -366,55 +383,55 @@
   <!-- =================================================== -->
   <!-- ros2_control hardware interface -->
-<ros2_control name="arm_system" type="system">
-  <hardware>
-    <plugin>gz_ros2_control/GazeboSimSystem</plugin>
-  </hardware>
-  <joint name="arm_base_joint">
-    <command_interface name="position"/>
-    <state_interface name="position"/>
-    <state_interface name="velocity"/>
-  </joint>
-  <joint name="upper_arm_joint">
-    <command_interface name="position"/>
-    <state_interface name="position">
-      <param name="initial_value">1.57</param>
-    </state_interface>
-    <state_interface name="velocity"/>
-  </joint>
-  <joint name="forearm_joint">
-    <command_interface name="position"/>
-    <state_interface name="position">
-      <param name="initial_value">-1.57</param>
-    </state_interface>
-    <state_interface name="velocity"/>
-  </joint>
-  <joint name="wrist_joint">
-    <command_interface name="position"/>
-    <state_interface name="position">
-      <param name="initial_value">-1.57</param>
-    </state_interface>
-    <state_interface name="velocity"/>
-  </joint>
-  <joint name="gripper_baseTOwrist_joint">
-    <command_interface name="position"/>
-    <state_interface name="position"/>
-    <state_interface name="velocity"/>
-  </joint>
-  <joint name="gripper_base_joint">
-    <command_interface name="position"/>
-    <state_interface name="position"/>
-    <state_interface name="velocity"/>
-  </joint>
-  <joint name="right_prong_joint">
-    <command_interface name="position"/>
-    <state_interface name="position"/>
-    <state_interface name="velocity"/>
-  </joint>
-  <joint name="left_prong_joint">
-    <command_interface name="position"/>
-    <state_interface name="position"/>
-    <state_interface name="velocity"/>
-  </joint>
-</ros2_control>
+  <ros2_control name="arm_system" type="system">
+    <hardware>
+      <plugin>gz_ros2_control/GazeboSimSystem</plugin>
+    </hardware>
+    <joint name="arm_base_joint">
+      <command_interface name="position"/>
+      <state_interface name="position"/>
+      <state_interface name="velocity"/>
+    </joint>
+    <joint name="upper_arm_joint">
+      <command_interface name="position"/>
+      <state_interface name="position">
+        <param name="initial_value">1.57</param>
+      </state_interface>
+      <state_interface name="velocity"/>
+    </joint>
+    <joint name="forearm_joint">
+      <command_interface name="position"/>
+      <state_interface name="position">
+        <param name="initial_value">-1.57</param>
+      </state_interface>
+      <state_interface name="velocity"/>
+    </joint>
+    <joint name="wrist_joint">
+      <command_interface name="position"/>
+      <state_interface name="position">
+        <param name="initial_value">-1.57</param>
+      </state_interface>
+      <state_interface name="velocity"/>
+    </joint>
+    <joint name="gripper_baseTOwrist_joint">
+      <command_interface name="position"/>
+      <state_interface name="position"/>
+      <state_interface name="velocity"/>
+    </joint>
+    <joint name="gripper_base_joint">
+      <command_interface name="position"/>
+      <state_interface name="position"/>
+      <state_interface name="velocity"/>
+    </joint>
+    <joint name="right_prong_joint">
+      <command_interface name="position"/>
+      <state_interface name="position"/>
+      <state_interface name="velocity"/>
+    </joint>
+    <joint name="left_prong_joint">
+      <command_interface name="position"/>
+      <state_interface name="position"/>
+      <state_interface name="velocity"/>
+    </joint>
+  </ros2_control>
   <!-- ==================== GAZEBO FRICTION & CONTACT PROPERTIES ==================== -->
   <gazebo reference="right_prong_link">
@@ -438,16 +455,22 @@
   <!-- Namespace for this arm instance (arm1 or arm2) -->
   <xacro:arg name="arm_namespace" default="arm1"/>
+  <xacro:property name="c_file" value="$(arg controllers_file)"/>
   <!-- gz_ros2_control plugin — each instance gets its own namespace so
        two arms can coexist with separate controller_managers -->
-  <gazebo>
-    <plugin filename="gz_ros2_control-system"
-            name="gz_ros2_control::GazeboSimROS2ControlPlugin">
-      <parameters>$(arg controllers_file)</parameters>
-      <robot_param>robot_description</robot_param>
-      <robot_param_node>arm_state_publisher</robot_param_node>
-      <ros>
-        <namespace>/$(arg arm_namespace)</namespace>
-      </ros>
-    </plugin>
-  </gazebo>
+  <xacro:if value="${c_file != ''}">
+    <gazebo>
+      <plugin filename="gz_ros2_control-system"
+              name="gz_ros2_control::GazeboSimROS2ControlPlugin">
+        <parameters>$(arg controllers_file)</parameters>
+        <robot_param>robot_description</robot_param>
+        <robot_param_node>arm_state_publisher</robot_param_node>
+        <ros>
+          <namespace>/$(arg arm_namespace)</namespace>
+        </ros>
+      </plugin>
+    </gazebo>
+  </xacro:if>
+  <xacro:unless value="${c_file != ''}">
+    <gazebo><static>true</static></gazebo>
+  </xacro:unless>
 </robot>

File: src/robot_description/urdf/robot.urdf.xacro (robot description, xacro)
@@ -32,4 +32,15 @@
          sfp_ctr      = cover_top_z + stdh + sfh/2= 0.045+0.052+0.005 = 0.102
   -->
+  <!-- Tray walls (funnel) mounted on standoff_floor.
+       Provide a 30 mm lip angled 15° outward to guide the delivery box to
+       centre even if the arm drops it up to ~50 mm off-centre.
+       wall_h   = 0.030  (lip height above floor top surface)
+       wall_t   = 0.006  (wall thickness)
+       tilt     = 15°    (0.5236 rad) outward on each wall
+       Joint z  = sfp_half_h + wall_half_h = 0.005 + 0.015 = 0.020
+  -->
+  <xacro:property name="tray_wall_h"    value="0.045"/>
+  <xacro:property name="tray_wall_t"    value="0.006"/>
+  <xacro:property name="tray_wall_mass" value="0.02"/>
   <!-- ==================== INERTIA MACROS ==================== -->
   <xacro:macro name="box_inertia" params="m x y z">
@@ -99,6 +110,10 @@
     </joint>
     <gazebo reference="${name}_wheel">
-      <mu1>0.8</mu1>
-      <mu2>0.05</mu2>
+      <!-- mu1/mu2 tuning for 4-fixed-wheel skid-steer:
+           mu2 too high -> bot cannot pivot (wheels scrub, chassis stalls);
+           mu2 too low  -> bot SLIDES sideways during turns (odometry lies).
+           0.3 = compromise: pivots with moderate scrub. Verified live. -->
+      <mu1>1.1</mu1>
+      <mu2>0.3</mu2>
       <kp>100000.0</kp>
       <kd>10.0</kd>
@@ -141,4 +156,39 @@
     </joint>
   </xacro:macro>
+  <!-- ==================== TRAY WALL MACRO ====================
+       A single retention lip fixed to standoff_floor.
+       params:
+         name        – unique suffix (front / rear / left / right)
+         wx / wy     – box dimensions in X and Y (one axis = tray_wall_t)
+         x_off/y_off – wall centre relative to standoff_floor centre
+         rpy         – outward tilt (15° = 0.5236 rad around relevant axis)
+       z joint = sfp_half_h + wall_half_h = 0.005 + 0.015 = 0.020
+  -->
+  <xacro:macro name="tray_wall" params="name wx wy x_off y_off rpy">
+    <link name="tray_wall_${name}">
+      <visual>
+        <origin xyz="0 0 0" rpy="0 0 0"/>
+        <geometry>
+          <box size="${wx} ${wy} ${tray_wall_h}"/>
+        </geometry>
+        <material name="orange_tray">
+          <color rgba="1.0 0.45 0.0 1"/>
+        </material>
+      </visual>
+      <collision>
+        <origin xyz="0 0 0" rpy="0 0 0"/>
+        <geometry>
+          <box size="${wx} ${wy} ${tray_wall_h}"/>
+        </geometry>
+      </collision>
+      <xacro:box_inertia m="${tray_wall_mass}" x="${wx}" y="${wy}" z="${tray_wall_h}"/>
+    </link>
+    <joint name="tray_wall_${name}_joint" type="fixed">
+      <parent link="standoff_floor"/>
+      <child  link="tray_wall_${name}"/>
+      <!-- z: sfp_half_h + wall_half_h = 0.005 + 0.015 = 0.020 -->
+      <origin xyz="${x_off} ${y_off} 0.020" rpy="${rpy}"/>
+    </joint>
+  </xacro:macro>
   <!-- ==================== BASE FOOTPRINT ==================== -->
   <link name="base_footprint"/>
@@ -252,4 +302,40 @@
     <origin xyz="0 0 0.062" rpy="0 0 0"/>
   </joint>
+  <!-- ==================== TRAY WALLS (4 retention lips on standoff_floor) ====================
+       standoff_floor: 0.35 m (X) × 0.25 m (Y) × 0.01 m (Z)
+       Height: 0.030 m  |  Tilt: 15° outward  |  Joint z = 0.020 (sfp_half + wall_half)
+       Front/rear walls span full Y width.  Left/right walls span inner X (fit between front/rear).
+       Tilt rotations (right-hand rule, outward = away from tray centre):
+         front (+X): pitch +0.5236   rear (−X): pitch −0.5236
+         left  (+Y): roll  −0.5236   right(−Y): roll  +0.5236
+  -->
+  <!-- Front wall: spans full Y width, sits at +X edge, top tilts outward (+X) -->
+  <xacro:tray_wall name="front"
+    wx="${tray_wall_t}"
+    wy="${standoff_floor_width}"
+    x_off="${standoff_floor_length/2 - tray_wall_t/2}"
+    y_off="0"
+    rpy="0 0.5236 0"/>
+  <!-- Rear wall: spans full Y width, sits at -X edge, top tilts outward (-X) -->
+  <xacro:tray_wall name="rear"
+    wx="${tray_wall_t}"
+    wy="${standoff_floor_width}"
+    x_off="${-(standoff_floor_length/2 - tray_wall_t/2)}"
+    y_off="0"
+    rpy="0 -0.5236 0"/>
+  <!-- Left wall: inner X span, sits at +Y edge, top tilts outward (+Y) -->
+  <xacro:tray_wall name="left"
+    wx="${standoff_floor_length - 2*tray_wall_t}"
+    wy="${tray_wall_t}"
+    x_off="0"
+    y_off="${standoff_floor_width/2 - tray_wall_t/2}"
+    rpy="-0.5236 0 0"/>
+  <!-- Right wall: inner X span, sits at -Y edge, top tilts outward (-Y) -->
+  <xacro:tray_wall name="right"
+    wx="${standoff_floor_length - 2*tray_wall_t}"
+    wy="${tray_wall_t}"
+    x_off="0"
+    y_off="${-(standoff_floor_width/2 - tray_wall_t/2)}"
+    rpy="0.5236 0 0"/>
   <!-- ==================== LIDAR ====================
        Mounts on top of cover_plate (centre of the plate).
