Commit message: Addition: added the forearm link and identified a bug that is causing the whole to rotate.

File: src/arm_description/urdf/arm.urdf.xacro (robot description, xacro)
@@ -2,5 +2,5 @@
 <robot name="arm" xmlns:xacro="http://www.ros.org/wiki/xacro">
   <!-- ==================== PROPERTIES ==================== -->
-  <xacro:property name="arm_base_link_height" value="0.01"/>
+  <xacro:property name="arm_base_link_height" value="0.02"/>
   <xacro:property name="arm_base_link_radius" value="0.05"/>
   <xacro:property name="arm_base_link_weight" value="0.3"/>
@@ -29,4 +29,10 @@
     </material>
   </visual>
+  <collision>
+    <origin xyz="0 0 0" rpy="0 0 0"/>
+    <geometry>
+      <cylinder radius="0.05" length="0.02"/>
+    </geometry>
+  </collision>
   <xacro:cylinder_inertia m="${arm_base_link_weight}" r="${arm_base_link_radius}" h="${arm_base_link_height}"/>
   </link>
@@ -34,7 +40,59 @@
     <parent link="arm_mount"/>
     <child link="arm_base_link"/>
-    <origin xyz="0.0 0 0.0275" rpy="0 0 0"/>
+    <origin xyz="0.0 0 0.0325" rpy="0 0 0"/>
     <limit lower="-3.14" upper="3.14" effort="10" velocity="1.0"/>
     <axis xyz="0 0 1"/>
   </joint>
+  <!-- ==================== FOREARM LINK ==================== -->
+  <link name="forearm_link">
+    <visual>
+      <origin xyz="0 0 0.065" rpy="0 1.5707 0"/>
+      <geometry>
+        <cylinder radius="0.022" length="0.13"/>
+      </geometry>
+      <material name="green">
+        <color rgba="0.035 0.85 0.035 1"/>
+      </material>
+    </visual>
+    <collision>
+      <origin xyz="0 0 0.065" rpy="0 1.5707 0"/>
+      <geometry>
+        <cylinder radius="0.022" length="0.13"/>
+      </geometry>
+    </collision>
+    <xacro:cylinder_inertia m="0.3" r="0.022" h="0.13"/>
+  </link>
+  <joint name="forearm_joint" type="revolute">
+    <parent link="upper_arm_link"/>
+    <child link="forearm_link"/>
+    <origin xyz="0 0 0.17" rpy="0 0 0"/>
+    <limit lower="-3.14" upper="3.14" effort="10" velocity="1.0"/>
+    <axis xyz="0 1 0"/>
+  </joint>
+  <!-- ==================== UPPER ARM LINK ==================== -->
+  <link name="upper_arm_link">
+    <visual>
+      <origin xyz="0 0 0.085" rpy="0 1.5707 0"/>
+      <geometry>
+        <cylinder radius="0.025" length="0.17"/>
+      </geometry>
+      <material name="blue">
+        <color rgba="0.035 0.035 0.85 1"/>
+      </material>
+    </visual>
+    <collision>
+      <origin xyz="0 0 0.085" rpy="0 1.5707 0"/>
+      <geometry>
+      <cylinder radius="0.025" length="0.17"/>
+      </geometry>
+    </collision>
+    <xacro:cylinder_inertia m="0.4" r="0.025" h="0.17"/>
+  </link>
+  <joint name="upper_arm_joint" type="revolute">
+    <parent link="arm_base_link"/>
+    <child link="upper_arm_link"/>
+    <origin xyz="0 0 0.01" rpy="0 0 0"/>
+    <limit lower="-3.14" upper="3.14" effort="10" velocity="1.0"/>
+    <axis xyz="0 1 0"/>
+  </joint>
 </robot>

File: src/robot_description/urdf/robot.urdf.xacro (robot description, xacro)
@@ -6,5 +6,5 @@
   <xacro:property name="base_width"  value="0.25"/>
   <xacro:property name="base_height" value="0.07"/>
-  <xacro:property name="base_mass"   value="2.5"/>
+  <xacro:property name="base_mass"   value="5.0"/>
   <xacro:property name="wheel_radius" value="0.05"/>
   <xacro:property name="wheel_width"  value="0.04"/>

Commit message: Addition: Added the wrist link to the arm.

File: src/arm_description/urdf/arm.urdf.xacro (robot description, xacro)
@@ -44,34 +44,8 @@
     <axis xyz="0 0 1"/>
   </joint>
-  <!-- ==================== FOREARM LINK ==================== -->
-  <link name="forearm_link">
-    <visual>
-      <origin xyz="0 0 0.065" rpy="0 1.5707 0"/>
-      <geometry>
-        <cylinder radius="0.022" length="0.13"/>
-      </geometry>
-      <material name="green">
-        <color rgba="0.035 0.85 0.035 1"/>
-      </material>
-    </visual>
-    <collision>
-      <origin xyz="0 0 0.065" rpy="0 1.5707 0"/>
-      <geometry>
-        <cylinder radius="0.022" length="0.13"/>
-      </geometry>
-    </collision>
-    <xacro:cylinder_inertia m="0.3" r="0.022" h="0.13"/>
-  </link>
-  <joint name="forearm_joint" type="revolute">
-    <parent link="upper_arm_link"/>
-    <child link="forearm_link"/>
-    <origin xyz="0 0 0.17" rpy="0 0 0"/>
-    <limit lower="-3.14" upper="3.14" effort="10" velocity="1.0"/>
-    <axis xyz="0 1 0"/>
-  </joint>
   <!-- ==================== UPPER ARM LINK ==================== -->
   <link name="upper_arm_link">
     <visual>
-      <origin xyz="0 0 0.085" rpy="0 1.5707 0"/>
+      <origin xyz="0 0 0.085" rpy="0 0 0"/>
       <geometry>
         <cylinder radius="0.025" length="0.17"/>
@@ -82,5 +56,5 @@
     </visual>
     <collision>
-      <origin xyz="0 0 0.085" rpy="0 1.5707 0"/>
+      <origin xyz="0 0 0.085" rpy="0 0 0"/>
       <geometry>
       <cylinder radius="0.025" length="0.17"/>
@@ -96,3 +70,93 @@
     <axis xyz="0 1 0"/>
   </joint>
+  <!-- ==================== FOREARM LINK ==================== -->
+  <link name="forearm_link">
+    <visual>
+      <origin xyz="0 0 0.065" rpy="0 0 0"/>
+      <geometry>
+        <cylinder radius="0.022" length="0.13"/>
+      </geometry>
+      <material name="green">
+        <color rgba="0.035 0.85 0.035 1"/>
+      </material>
+    </visual>
+    <collision>
+      <origin xyz="0 0 0.065" rpy="0 0 0"/>
+      <geometry>
+        <cylinder radius="0.022" length="0.13"/>
+      </geometry>
+    </collision>
+    <xacro:cylinder_inertia m="0.3" r="0.022" h="0.13"/>
+  </link>
+  <joint name="forearm_joint" type="revolute">
+    <parent link="upper_arm_link"/>
+    <child link="forearm_link"/>
+    <origin xyz="0 0 0.17" rpy="0 1.5707 0"/>
+    <limit lower="-3.14" upper="3.14" effort="10" velocity="1.0"/>
+    <axis xyz="0 1 0"/>
+  </joint>
+<!-- ==================== WRIST LINK ==================== -->
+  <link name = "wrist_link">
+    <visual>
+      <origin xyz="0.05 0 0" rpy="0 0 0"/>
+      <geometry>
+        <cylinder radius="0.02" length="0.1"/>
+      </geometry>
+      <material name="red">
+        <color rgba="0.85 0.035 0.035 1"/>
+      </material>
+    </visual>
+    <collision>
+      <origin xyz="0.05 0 0" rpy="0 0 0"/>
+      <geometry>
+        <cylinder radius="0.02" length="0.1"/>
+      </geometry>
+    </collision>
+    <xacro:cylinder_inertia m="0.2" r="0.02" h="0.1"/>
+  </link>
+  <joint name="wrist_joint" type="revolute">
+    <parent link="forearm_link"/>
+    <child link="wrist_link"/>
+    <origin xyz="0.13 0 0" rpy="0 0 0"/>
+    <limit lower="-3.14" upper="3.14" effort="10" velocity="1.0"/>
+    <axis xyz="1 0 0"/>
+  </joint>
+<!-- =================================================== -->
+<gazebo>
+  <plugin filename="gz-sim-joint-state-publisher-system"
+          name="gz::sim::systems::JointStatePublisher">
+  </plugin>
+  <plugin filename="gz-sim-joint-position-controller-system"
+          name="gz::sim::systems::JointPositionController">
+    <joint_name>upper_arm_joint</joint_name>
+    <p_gain>10</p_gain>
+    <i_gain>0.1</i_gain>
+    <d_gain>0.01</d_gain>
+    <initial_position>0.0</initial_position>
+  </plugin>
+  <plugin filename="gz-sim-joint-position-controller-system"
+          name="gz::sim::systems::JointPositionController">
+    <joint_name>forearm_joint</joint_name>
+    <p_gain>10</p_gain>
+    <i_gain>0.1</i_gain>
+    <d_gain>0.01</d_gain>
+    <initial_position>0.0</initial_position>
+  </plugin>
+  <plugin filename="gz-sim-joint-position-controller-system"
+          name="gz::sim::systems::JointPositionController">
+    <joint_name>arm_base_joint</joint_name>
+    <p_gain>10</p_gain>
+    <i_gain>0.1</i_gain>
+    <d_gain>0.01</d_gain>
+    <initial_position>0.0</initial_position>
+  </plugin>
+  <plugin filename="gz-sim-joint-position-controller-system"
+          name="gz::sim::systems::JointPositionController">
+    <joint_name>wrist_joint</joint_name>
+    <p_gain>10</p_gain>
+    <i_gain>0.1</i_gain>
+    <d_gain>0.01</d_gain>
+    <initial_position>0.0</initial_position>
+  </plugin>
+</gazebo>
 </robot>

Commit message: Arm Completion: Completed the arm xacro file with few tweaks reamaining

File: src/arm_description/urdf/arm.urdf.xacro (robot description, xacro)
@@ -6,4 +6,5 @@
   <xacro:property name="arm_base_link_weight" value="0.3"/>
   <!-- ==================== Inertia Macros ================ -->
+  <!-- Cylinder Inertia -->
   <xacro:macro name="cylinder_inertia" params="m r h">
     <inertial>
@@ -18,4 +19,30 @@
     </inertial>
   </xacro:macro>
+  <!--Sphere Inertia -->
+  <xacro:macro name="sphere_inertia" params="m r">
+    <inertial>
+      <origin xyz="0 0 0" rpy="0 0 0"/>
+      <mass value="${m}"/>
+      <inertia
+        ixx="${(2/5)*m*r*r}"
+        ixy="0" ixz="0"
+        iyy="${(2/5)*m*r*r}"
+        iyz="0"
+        izz="${(2/5)*m*r*r}"/>
+    </inertial>
+  </xacro:macro>
+  <!-- Box Inertia -->
+  <xacro:macro name="box_inertia" params="m x y z">
+    <inertial>
+      <origin xyz="0 0 0" rpy="0 0 0"/>
+      <mass value="${m}"/>
+      <inertia
+        ixx="${(1/12)*m*(y*y+z*z)}"
+        ixy="0" ixz="0"
+        iyy="${(1/12)*m*(x*x+z*z)}"
+        iyz="0"
+        izz="${(1/12)*m*(x*x+y*y)}"/>
+    </inertial>
+  </xacro:macro>
   <!-- ==================== ARM BASE LINK ==================== -->
   <link name="arm_base_link">
@@ -61,5 +88,5 @@
       </geometry>
     </collision>
-    <xacro:cylinder_inertia m="0.4" r="0.025" h="0.17"/>
+    <xacro:cylinder_inertia m="1.0" r="0.025" h="0.17"/>
   </link>
   <joint name="upper_arm_joint" type="revolute">
@@ -70,4 +97,30 @@
     <axis xyz="0 1 0"/>
   </joint>
+  <!-- ==================== UPPER-FORE ARM LINK ==================== -->
+  <link name="upper_forearm_link">
+    <visual>
+      <origin xyz="0 0 0" rpy="0 0 0"/>
+      <geometry>
+        <sphere radius="0.0375"/>
+      </geometry>
+      <material name="cyan">
+        <color rgba="0.035 0.85 0.85 1"/>
+      </material>
+    </visual>
+    <collision>
+      <origin xyz="0 0 0" rpy="0 0 0"/>
+      <geometry>
+        <sphere radius="0.025"/>
+      </geometry>
+    </collision>
+    <xacro:sphere_inertia m="0.3" r="0.025"/>
+  </link>
+  <joint name="upper_forearm_joint" type="fixed">
+    <parent link="upper_arm_link"/>
+    <child link="upper_forearm_link"/>
+    <origin xyz="0 0 0.17" rpy="0 1.5707 0"/>
+    <limit lower="-3.14" upper="3.14" effort="10" velocity="1.0"/>
+    <axis xyz="0 1 0"/>
+  </joint>
   <!-- ==================== FOREARM LINK ==================== -->
   <link name="forearm_link">
@@ -96,8 +149,34 @@
     <axis xyz="0 1 0"/>
   </joint>
+  <!-- ==================== FOREARM-WRIST LINK ==================== -->
+  <link name="forearm_wrist_link">
+    <visual>
+      <origin xyz="0 0 0" rpy="0 0 0"/>
+      <geometry>
+        <sphere radius="0.0375"/>
+      </geometry>
+      <material name="cyan">
+        <color rgba="0.035 0.85 0.85 1"/>
+      </material>
+    </visual>
+    <collision>
+      <origin xyz="0 0 0" rpy="0 0 0"/>
+      <geometry>
+        <sphere radius="0.025"/>
+      </geometry>
+    </collision>
+    <xacro:sphere_inertia m="0.3" r="0.025"/>
+  </link>
+  <joint name="forearm_wrist_joint" type="fixed">
+    <parent link="forearm_link"/>
+    <child link="forearm_wrist_link"/>
+    <origin xyz="0 0 0.13" rpy="0 0 0"/>
+    <limit lower="-3.14" upper="3.14" effort="10" velocity="1.0"/>
+    <axis xyz="0 1 0"/>
+  </joint>
 <!-- ==================== WRIST LINK ==================== -->
   <link name = "wrist_link">
     <visual>
-      <origin xyz="0.05 0 0" rpy="0 0 0"/>
+      <origin xyz="0 0 0.05" rpy="0 0 0"/>
       <geometry>
         <cylinder radius="0.02" length="0.1"/>
@@ -108,5 +187,5 @@
     </visual>
     <collision>
-      <origin xyz="0.05 0 0" rpy="0 0 0"/>
+      <origin xyz="0 0 0.05" rpy="0 0 0"/>
       <geometry>
         <cylinder radius="0.02" length="0.1"/>
@@ -118,8 +197,111 @@
     <parent link="forearm_link"/>
     <child link="wrist_link"/>
-    <origin xyz="0.13 0 0" rpy="0 0 0"/>
+    <origin xyz="0 0 0.13" rpy="-1.5707 0 0"/>
     <limit lower="-3.14" upper="3.14" effort="10" velocity="1.0"/>
     <axis xyz="1 0 0"/>
   </joint>
+<!-- ==================== GRIPPER_BASE_TO_WRIST LINK ==================== -->
+  <link name="gripper_baseTOwrist_link">
+    <visual>
+      <origin xyz="0 0 0" rpy="0 0 0"/>
+      <geometry>
+        <cylinder radius="0.008" length="0.01"/>
+      </geometry>
+      <material name="cyan">
+        <color rgba="0.035 0.85 0.85 1"/>
+      </material>
+    </visual>
+    <collision>
+      <origin xyz="0 0 0" rpy="0 0 0"/>
+      <geometry>
+        <cylinder radius="0.008" length="0.01"/>
+      </geometry>
+    </collision>
+    <xacro:cylinder_inertia m="0.2" r="0.008" h="0.01"/>
+  </link>
+  <joint name="gripper_baseTOwrist_joint" type="fixed">
+    <parent link="wrist_link"/>
+    <child link="gripper_baseTOwrist_link"/>
+    <origin xyz="0 0 0.1" rpy="0 0 0"/>
+    <limit lower="-3.14" upper="3.14" effort="10" velocity="1.0"/>
+    <axis xyz="0 1 0"/>
+  </joint>
+<!-- ==================== GRIPPER BASE LINK ==================== -->
+  <link name="gripper_base_link">
+    <visual>
+      <origin xyz="0 0 0" rpy="0 0 0"/>
+      <geometry>
+        <box size="0.008 0.04 0.04"/>
+      </geometry>
+      <material name="cyan">
+        <color rgba="0.035 0.85 0.85 1"/>
+      </material>
+    </visual>
+    <collision>
+      <origin xyz="0 0 0" rpy="0 0 0"/>
+      <geometry>
+        <box size="0.008 0.04 0.04"/>
+      </geometry>
+    </collision>
+    <xacro:box_inertia m="0.2" x="0.008" y="0.04" z="0.04"/>
+  </link>
+  <joint name="gripper_base_joint" type="fixed">
+    <parent link="gripper_baseTOwrist_link"/>
+    <child link="gripper_base_link"/>
+    <origin xyz="0 0 0.005" rpy="0 0 0"/>
+  </joint>
+<!-- ==================== PRONGS ==================== -->
+<!--RIGHT PRONG-->
+<link name="right_prong_link">
+  <visual>
+    <origin xyz="0 0 0" rpy="0 0 0"/>
+    <geometry>
+      <box size="0.02 0.005 0.06"/>
+    </geometry>
+    <material name="cyan">
+      <color rgba="0.035 0.85 0.85 1"/>
+    </material>
+  </visual>
+  <collision>
+    <origin xyz="0 0 0" rpy="0 0 0"/>
+    <geometry>
+      <box size="0.02 0.005 0.06"/>
+    </geometry>
+  </collision>
+  <xacro:box_inertia m="0.05" x="0.02" y="0.005" z="0.06"/>
+</link>
+<joint name="right_prong_joint" type="prismatic">
+  <parent link="gripper_base_link"/>
+  <child link="right_prong_link"/>
+  <origin xyz="0 0.02 0" rpy="0 0 0"/>
+  <limit lower="0" upper="0.08" effort="10" velocity="1.0"/>
+  <axis xyz="0 1 0"/>
+</joint>
+<!--LEFT PRONG-->
+<link name="left_prong_link">
+  <visual>
+    <origin xyz="0 0 0" rpy="0 0 0"/>
+    <geometry>
+      <box size="0.02 0.005 0.06"/>
+    </geometry>
+    <material name="cyan">
+      <color rgba="0.035 0.85 0.85 1"/>
+    </material>
+  </visual>
+  <collision>
+    <origin xyz="0 0 0" rpy="0 0 0"/>
+    <geometry>
+      <box size="0.02 0.005 0.06"/>
+    </geometry>
+  </collision>
+  <xacro:box_inertia m="0.05" x="0.02" y="0.005" z="0.06"/>
+</link>
+<joint name="left_prong_joint" type="prismatic">
+  <parent link="gripper_base_link"/>
+  <child link="left_prong_link"/>
+  <origin xyz="0 -0.02 0" rpy="0 0 0"/>
+  <limit lower="-0.08" upper="0" effort="10" velocity="1.0"/>
+  <axis xyz="0 1 0"/>
+</joint>
 <!-- =================================================== -->
 <gazebo>
@@ -131,4 +313,44 @@
     <joint_name>upper_arm_joint</joint_name>
     <p_gain>10</p_gain>
+    <i_gain>1.0</i_gain>
+    <d_gain>5.0</d_gain>
+    <initial_position>0.0</initial_position>
+  </plugin>
+  <plugin filename="gz-sim-joint-position-controller-system"
+          name="gz::sim::systems::JointPositionController">
+    <joint_name>forearm_joint</joint_name>
+    <p_gain>10</p_gain>
+    <i_gain>1.0</i_gain>
+    <d_gain>5.0</d_gain>
+    <initial_position>0.0</initial_position>
+  </plugin>
+  <plugin filename="gz-sim-joint-position-controller-system"
+          name="gz::sim::systems::JointPositionController">
+    <joint_name>arm_base_joint</joint_name>
+    <p_gain>10</p_gain>
+    <i_gain>1.0</i_gain>
+    <d_gain>5.0</d_gain>
+    <initial_position>0.0</initial_position>
+  </plugin>
+  <plugin filename="gz-sim-joint-position-controller-system"
+          name="gz::sim::systems::JointPositionController">
+    <joint_name>wrist_joint</joint_name>
+    <p_gain>10</p_gain>
+    <i_gain>1.0</i_gain>
+    <d_gain>5.0</d_gain>
+    <initial_position>0.0</initial_position>
+  </plugin>
+  <plugin filename="gz-sim-joint-position-controller-system"
+          name="gz::sim::systems::JointPositionController">
+    <joint_name>gripper_baseTOwrist_joint</joint_name>
+    <p_gain>10</p_gain>
+    <i_gain>1.0</i_gain>
+    <d_gain>5.0</d_gain>
+    <initial_position>0.0</initial_position>
+  </plugin>
+  <plugin filename="gz-sim-joint-position-controller-system"
+          name="gz::sim::systems::JointPositionController">
+    <joint_name>right_prong_joint</joint_name>
+    <p_gain>10</p_gain>
     <i_gain>0.1</i_gain>
     <d_gain>0.01</d_gain>
@@ -137,5 +359,5 @@
   <plugin filename="gz-sim-joint-position-controller-system"
           name="gz::sim::systems::JointPositionController">
-    <joint_name>forearm_joint</joint_name>
+    <joint_name>left_prong_joint</joint_name>
     <p_gain>10</p_gain>
     <i_gain>0.1</i_gain>
@@ -143,20 +365,4 @@
     <initial_position>0.0</initial_position>
   </plugin>
-  <plugin filename="gz-sim-joint-position-controller-system"
-          name="gz::sim::systems::JointPositionController">
-    <joint_name>arm_base_joint</joint_name>
-    <p_gain>10</p_gain>
-    <i_gain>0.1</i_gain>
-    <d_gain>0.01</d_gain>
-    <initial_position>0.0</initial_position>
-  </plugin>
-  <plugin filename="gz-sim-joint-position-controller-system"
-          name="gz::sim::systems::JointPositionController">
-    <joint_name>wrist_joint</joint_name>
-    <p_gain>10</p_gain>
-    <i_gain>0.1</i_gain>
-    <d_gain>0.01</d_gain>
-    <initial_position>0.0</initial_position>
-  </plugin>
 </gazebo>
 </robot>

Commit message: Add arm_teleop controller, joint bridge congig for arm links, the arm is working now.

File: src/arm_description/urdf/arm.urdf.xacro (robot description, xacro)
@@ -255,5 +255,5 @@
 <link name="right_prong_link">
   <visual>
-    <origin xyz="0 0 0" rpy="0 0 0"/>
+    <origin xyz="0 0 0.018" rpy="0 0 0"/>
     <geometry>
       <box size="0.02 0.005 0.06"/>
@@ -264,5 +264,5 @@
   </visual>
   <collision>
-    <origin xyz="0 0 0" rpy="0 0 0"/>
+    <origin xyz="0 0 0.018" rpy="0 0 0"/>
     <geometry>
       <box size="0.02 0.005 0.06"/>
@@ -274,5 +274,5 @@
   <parent link="gripper_base_link"/>
   <child link="right_prong_link"/>
-  <origin xyz="0 0.02 0" rpy="0 0 0"/>
+  <origin xyz="0 0.02 0.018" rpy="0 0 0"/>
   <limit lower="0" upper="0.08" effort="10" velocity="1.0"/>
   <axis xyz="0 1 0"/>
@@ -281,5 +281,5 @@
 <link name="left_prong_link">
   <visual>
-    <origin xyz="0 0 0" rpy="0 0 0"/>
+    <origin xyz="0 0 0.018" rpy="0 0 0"/>
     <geometry>
       <box size="0.02 0.005 0.06"/>
@@ -290,5 +290,5 @@
   </visual>
   <collision>
-    <origin xyz="0 0 0" rpy="0 0 0"/>
+    <origin xyz="0 0 0.018" rpy="0 0 0"/>
     <geometry>
       <box size="0.02 0.005 0.06"/>
@@ -300,5 +300,5 @@
   <parent link="gripper_base_link"/>
   <child link="left_prong_link"/>
-  <origin xyz="0 -0.02 0" rpy="0 0 0"/>
+  <origin xyz="0 -0.02 0.018" rpy="0 0 0"/>
   <limit lower="-0.08" upper="0" effort="10" velocity="1.0"/>
   <axis xyz="0 1 0"/>
@@ -353,6 +353,6 @@
     <joint_name>right_prong_joint</joint_name>
     <p_gain>10</p_gain>
-    <i_gain>0.1</i_gain>
-    <d_gain>0.01</d_gain>
+    <i_gain>1.0</i_gain>
+    <d_gain>5.0</d_gain>
     <initial_position>0.0</initial_position>
   </plugin>
@@ -361,6 +361,6 @@
     <joint_name>left_prong_joint</joint_name>
     <p_gain>10</p_gain>
-    <i_gain>0.1</i_gain>
-    <d_gain>0.01</d_gain>
+    <i_gain>1.0</i_gain>
+    <d_gain>5.0</d_gain>
     <initial_position>0.0</initial_position>
   </plugin>

Commit message: Minor updates

File: src/arm_description/urdf/arm.urdf.xacro (robot description, xacro)
@@ -145,5 +145,5 @@
     <parent link="upper_arm_link"/>
     <child link="forearm_link"/>
-    <origin xyz="0 0 0.17" rpy="0 1.5707 0"/>
+    <origin xyz="0 0 0.17" rpy="0 0 0"/>
     <limit lower="-3.14" upper="3.14" effort="10" velocity="1.0"/>
     <axis xyz="0 1 0"/>
@@ -257,5 +257,5 @@
     <origin xyz="0 0 0.018" rpy="0 0 0"/>
     <geometry>
-      <box size="0.02 0.005 0.06"/>
+      <box size="0.02 0.005 0.1"/>
     </geometry>
     <material name="cyan">
@@ -266,8 +266,8 @@
     <origin xyz="0 0 0.018" rpy="0 0 0"/>
     <geometry>
-      <box size="0.02 0.005 0.06"/>
+      <box size="0.02 0.005 0.1"/>
     </geometry>
   </collision>
-  <xacro:box_inertia m="0.05" x="0.02" y="0.005" z="0.06"/>
+  <xacro:box_inertia m="0.05" x="0.02" y="0.015" z="0.1"/>
 </link>
 <joint name="right_prong_joint" type="prismatic">
@@ -283,5 +283,5 @@
     <origin xyz="0 0 0.018" rpy="0 0 0"/>
     <geometry>
-      <box size="0.02 0.005 0.06"/>
+      <box size="0.02 0.005 0.1"/>
     </geometry>
     <material name="cyan">
@@ -292,8 +292,8 @@
     <origin xyz="0 0 0.018" rpy="0 0 0"/>
     <geometry>
-      <box size="0.02 0.005 0.06"/>
+      <box size="0.02 0.005 0.1"/>
     </geometry>
   </collision>
-  <xacro:box_inertia m="0.05" x="0.02" y="0.005" z="0.06"/>
+  <xacro:box_inertia m="0.05" x="0.02" y="0.015" z="0.1"/>
 </link>
 <joint name="left_prong_joint" type="prismatic">
@@ -323,5 +323,5 @@
     <i_gain>1.0</i_gain>
     <d_gain>5.0</d_gain>
-    <initial_position>0.0</initial_position>
+    <initial_position>1.5707</initial_position>
   </plugin>
   <plugin filename="gz-sim-joint-position-controller-system"
@@ -365,4 +365,16 @@
     <initial_position>0.0</initial_position>
   </plugin>
+</gazebo>
+<gazebo reference="right_prong_link">
+  <mu1>10.0</mu1>
+  <mu2>10.0</mu2>
+  <kp>1000000.0</kp>
+  <kd>1.0</kd>
+</gazebo>
+<gazebo reference="left_prong_link">
+  <mu1>10.0</mu1>
+  <mu2>10.0</mu2>
+  <kp>1000000.0</kp>
+  <kd>1.0</kd>
 </gazebo>
 </robot>
